File: our-programmer/esp32_programmer.sch (EAGLE design)
At the start: 59 parts, among them J16 10103592-0001LF-EK, Q1 MMBT3904_R1, Q2 MMBT3904_R1, U1 CP2102N-A02-GQFN24QFN24_CP210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, U2 AP2111H-3.3TRG1SOT-223_DIO-M, U3 NPN: BC817, U4 NPN: BC817, U5 NPN: BC817, U6 NPN: BC817

Commit message: Programmer board complete
Parts:
- added TP1, TP2, TP3: TEST-POINT3X5, SparkFun-Connectors:TEST-POINT3X5
Connections:
- net GND1 renamed BLEP3
- net GND2 renamed BLEP4
- net GND3 renamed BLEP1
- net GND4 renamed BLEP2
- removed net N$2: C1.1
- removed net N$3: C1.2, S2.2
- net EN_SEL: now also TP2.1
- net GND: now also C1.2, S2.2, TP3.1
- net IO0_SEL: now also TP1.1
- net VCC: now also C1.1
Other:
- moved on the sheet: C2, C3, J1, J4, TP12, TP13, TP14, TP26, TP27, TP35, U2
