File: esp32/esp32-kitchensink.brd (EAGLE design)
At the start: 100 x 80 mm, 189 parts, among them J14 MEM2075-00-140-01-A, J3 10103592-0001LF, Q1 MMBT3904_R1, Q2 MMBT3904_R1, Q3 AO3401, Q4 PN2222A-SOT-23, Q5 IRF7341TRPBF, U1 ESP32-WROOM-32D, U10 AH1807-W-7SC59_DIO-M, U11 DS3231M+TRL21-0042B_16_MXM-M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

Commit message: Added DC in and 5V regulator, Started initial pcb layout and routing
Parts:
- removed S3: JS102011JCQN, JS102011JCQN:SW_JS102011JCQN
- added C21: 0.47 uF, standardparts:1206
- added C22: 22 uF, standardparts:1206
- added C23: 1000 uF, rcl:140CLH-1010
- added D14: RS1BB-13-FSMA_DIO-M, UltraLibrarianParts:SMA_DIO-M
- added J16: 10103592-0001LF-EK, UltraLibrarianParts:AMPHENOL_10103592-0001LF
- added J17: (no value), SparkFun-Connectors:1X03_LONGPADS
- added J18: (no value), SparkFun-Connectors:1X03
- added J19: PJ-102AH, UltraLibrarianParts:CUI_PJ-102AH
- added S5: EG1224, UltraLibrarianParts:SW_EG1224
- added TP64, TP65: TP, UltraLibrarianParts:TP
- added TP66, TP67: TEST-POINT3X5, SparkFun-Connectors:PAD.03X.05
- added U9: TS2940CW50_RPG, UltraLibrarianParts:VREG_TS2940CW50_RPG
- J3: value 10103592-0001LF -> (none); device 10103592-0001LF:AMPHENOL_10103592-0001LF -> SparkFun-Connectors:1X03_LONGPADS
- moved H1 1124.6 mm to (134.1, 83.9)
- moved H3 1099.8 mm to (4.06, 84.8)
- moved H2 1051.7 mm to (134.6, 4.83)
- moved H4 1022.2 mm to (4.06, 4.06)
- moved TP1 329.7 mm to (213.4, -132.1)
- moved TP2 329.7 mm to (224.8, -132.1)
- moved TP3 329.7 mm to (213.4, -124.5)
- moved TP4 329.7 mm to (224.8, -124.5)
- moved TP5 329.7 mm to (213.4, -116.8)
- moved TP6 329.7 mm to (224.8, -116.8)
- moved C5 327.3 mm to (-36.8, -121.9)
- moved C6 327.3 mm to (-30.5, -121.9)
- moved CN2 327.3 mm to (-43.2, -120.7)
- moved D3 327.3 mm to (-44.5, -113.0)
- moved R10 327.3 mm to (-17.8, -121.9)
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Connections:
- removed net VOUT: C4.2, D4.1, Q3.2, S3.2
- new net 5V_DC_IN: C22.2, C23.+, J18.1, TP64.P$1, TP67.P$1, U9.3
- new net CP_RX: J17.3, TP20.P$1, U3.20
- new net CP_TX: J3.3, TP19.P$1, U3.21
- new net DC_JACK: D14.2, J19.1, TP65.P$1, TP66.P$1
- new net FTDI_RX: J1.2, J17.1, TP14.P$1
- new net FTDI_TX: J1.3, J3.1, TP13.P$1
- new net N$32: C21.2, U9.1
- new net N$43: C21.1, D14.1
- new net OFF: S5.3
- new net PWR_INPUT: J18.2, S5.2
- new net PWR_ON: D4.2, Q3.1, R8.1, S5.1, TP21.P$1
- net GND: now also C22.1, C23.-, J16.5, J19.2, J19.3, U9.2, U9.4; no longer J3.5
- net I2C_SCL: no longer TP58.P$1
- net I2C_SDA: now also TP58.P$1
- net N$5: now also J16.3; no longer J3.3
- net N$6: now also J16.2; no longer J3.2
- net RX: now also J17.2; no longer J1.2, TP14.P$1, TP20.P$1, U3.20
- net SHIELD: now also J16.P1, J16.P2, J16.P3, J16.P4, J16.P5, J16.P6; no longer J3.P1, J3.P2, J3.P3, J3.P4, J3.P5, J3.P6
- net TX: now also J3.2; no longer J1.3, TP13.P$1, TP19.P$1, U3.21
- net VIN: now also C4.2, D4.1, Q3.2; no longer S3.1
- net V_USB: now also J16.1, J18.3; no longer D4.2, J3.1, Q3.1, R8.1, TP21.P$1
Routing:
- net GND: track 0.00 -> 298.4 mm
- net VCC: track 0.00 -> 142.6 mm
- net 5V: track 0.00 -> 53.1 mm
- net I2C_SDA: track 0.00 -> 49.8 mm
- net 5V_DC_IN: track 0.00 -> 47.3 mm
- net I2C_SCL: track 0.00 -> 43.6 mm
- net VIN: track 0.00 -> 41.1 mm
- net CP_TX: track 0.00 -> 28.6 mm
- net CP_RX: track 0.00 -> 27.9 mm
- net PWR_ON: track 0.00 -> 27.5 mm
- net N$33: track 0.00 -> 26.6 mm
- net DC_JACK: track 0.00 -> 26.5 mm
- net V_BATT: track 0.00 -> 19.2 mm
- net FTDI_TX: track 0.00 -> 17.4 mm
- net N$5: track 0.00 -> 17.3 mm
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Other:
- board size 100 x 80 mm -> 139.4 x 88.9 mm
- board text added: "5V Regulator"

Commit message: Updates to larger kitchen sink files
Parts:
- moved R26 100.1 mm to (128.7, 31.6)
- moved R25 93.4 mm to (124.8, 31.6)
- moved R33 30.1 mm to (136.3, 68.7), turned to 270 degrees
- moved R34 28.9 mm to (133.7, 68.7), turned to 270 degrees
- moved R35 28.5 mm to (128.7, 68.8), turned to 270 degrees
- moved R37 28.3 mm to (123.6, 69.0), turned to 90 degrees
- moved TP14 21.8 mm to (98.3, 10.4)
- moved TP19 21.3 mm to (86.4, 20.6)
- moved R36 20.1 mm to (120.8, 69.0), turned to 90 degrees
- moved BT1 19.3 mm to (95.0, 53.0), flipped to the top
- moved TP20 19.0 mm to (86.4, 17.1)
- moved TP13 18.8 mm to (98.3, 12.4)
- moved J15 17.2 mm to (121.0, 63.0), turned to 0 degrees
- moved TP62 16.1 mm to (77.1, 28.1)
- moved TP63 15.3 mm to (78.9, 28.1)
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Connections:
- removed net CD: J14.P9, J15.1, R33.2
- new net SPI_CD: J14.P9, J15.7, R33.2
- net GND: now also J15.5; no longer J15.6
- net SPI_MISO: now also J15.6; no longer J15.2
- net SPI_MOSI: now also J15.2; no longer J15.3
- net SPI_SS: now also J15.1; no longer J15.5
- net VCC: now also J15.3; no longer J15.7
Routing:
- net VCC: track 142.6 -> 521.4 mm, vias 0 -> 12
- net GND: track 298.4 -> 166.6 mm
- net 5V_DC_IN: track 47.3 -> 84.8 mm, vias 0 -> 1
- net SPI_CD: track 0.00 -> 35.9 mm
- net V_USB: track 16.3 -> 49.9 mm, vias 0 -> 1
- net SPI_MISO: track 0.00 -> 31.2 mm
- net SPI_SCLK: track 0.00 -> 23.9 mm
- net SPI_MOSI: track 0.00 -> 20.8 mm
- net FTDI_TX: track 17.4 -> 38.1 mm
- net SPI_SS: track 0.00 -> 19.9 mm
- net EN: track 0.00 -> 15.9 mm
- net N$6: track 15.5 -> 27.2 mm
- net N$3: track 0.00 -> 11.1 mm
- net I2C_SDA: track 49.8 -> 39.9 mm
- net I2C_SCL: track 43.6 -> 34.4 mm
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