File: esp32/esp32-kitchensink.sch (EAGLE design)
At the start: 189 parts, among them J14 MEM2075-00-140-01-A, J3 10103592-0001LF, Q1 MMBT3904_R1, Q2 MMBT3904_R1, Q3 AO3401, Q4 PN2222A-SOT-23, Q5 IRF7341TRPBF, U1 ESP32-WROOM-32D, U10 AH1807-W-7SC59_DIO-M, U11 DS3231M+TRL21-0042B_16_MXM-M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

Commit message: Added DC in and 5V regulator, Started initial pcb layout and routing
Parts:
- removed S3: JS102011JCQN, JS102011JCQN:JS102011JCQN
- added C21: 0.47 uF, standardparts:CAPACITOR.1206
- added C22: 22 uF, standardparts:CAPACITOR.1206
- added C23: 1000 uF, rcl:CPOL-EU140CLH-1010
- added D14: RS1BB-13-FSMA_DIO-M, UltraLibrarianParts:RS1BB-13-FSMA_DIO-M
- added J16: 10103592-0001LF-EK, UltraLibrarianParts:10103592-0001LF-EK
- added J17: (no value), SparkFun-Connectors:CONN_03LONGPADS
- added J18: (no value), SparkFun-Connectors:CONN_03
- added J19: PJ-102AH, UltraLibrarianParts:PJ-102AH
- added S5: EG1224, UltraLibrarianParts:EG1224
- added TP64, TP65: TP, UltraLibrarianParts:TP
- added TP66, TP67: TEST-POINT3X5, SparkFun-Connectors:TEST-POINT3X5
- added U9: TS2940CW50_RPG, UltraLibrarianParts:TS2940CW50_RPG
- J3: value 10103592-0001LF -> (none); device 10103592-0001LF:10103592-0001LF -> SparkFun-Connectors:CONN_03LONGPADS
Connections:
- removed net VOUT: C4.2, D4.1, Q3.S, S3.2
- new net 5V_DC_IN: C22.2, C23.+, J18.1, TP64.P$1, TP67.1, U9.OUT
- new net CP_RX: J17.3, TP20.1, U3.RXD
- new net CP_TX: J3.3, TP19.1, U3.TXD
- new net DC_JACK: D14.2, J19.1, TP65.P$1, TP66.1
- new net FTDI_RX: J1.2, J17.1, TP14.1
- new net FTDI_TX: J1.3, J3.1, TP13.1
- new net N$32: C21.2, U9.IN
- new net N$43: C21.1, D14.1
- new net OFF: S5.3
- new net PWR_INPUT: J18.2, S5.2
- new net PWR_ON: D4.2, Q3.G, R8.1, S5.1, TP21.1
- net GND: now also C22.1, C23.-, J16.GND, J19.2, J19.3, U9.GND; no longer J3.GND
- net I2C_SCL: no longer TP58.1
- net I2C_SDA: now also TP58.1
- net N$5: now also J16.D+; no longer J3.D+
- net N$6: now also J16.D-; no longer J3.D-
- net RX: now also J17.2; no longer J1.2, TP14.1, TP20.1, U3.RXD
- net TX: now also J3.2; no longer J1.3, TP13.1, TP19.1, U3.TXD
- net VIN: now also C4.2, D4.1, Q3.S; no longer S3.1
- net V_USB: now also J16.VDD, J18.3; no longer D4.2, J3.VDD, Q3.G, R8.1, TP21.1
Other:
- note added: "I_o = 1 A"
- note added: "Input Selection"
- note added: "Power 2/3"
- note added: "Regulator"
- note added: "TS2940CW50 RPG Max Vin = 26 V"

Commit message: Updates to larger kitchen sink files
Connections:
- removed net CD: J14.CD, J15.1, R33.2
- new net SPI_CD: J14.CD, J15.7, R33.2
- net GND: now also J15.5; no longer J15.6
- net SPI_MISO: now also J15.6; no longer J15.2
- net SPI_MOSI: now also J15.2; no longer J15.3
- net SPI_SS: now also J15.1; no longer J15.5
- net VCC: now also J15.3; no longer J15.7
Changed lines of the file:
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@@
 <part name="SUPPLY22" library="SparkFun-PowerSymbols" library_urn="urn:adsk.eagle:library:530" deviceset="VCC" device=""/>
 <part name="J15" library="SparkFun-Connectors" library_urn="urn:adsk.eagle:library:513" deviceset="CONN_07" device="LONGPADS" package3d_urn="urn:adsk.eagle:package:38135/1"/>
-<part name="GND52" library="SparkFun-PowerSymbols" library_urn="urn:adsk.eagle:library:530" deviceset="GND" device=""/>
-<part name="SUPPLY20" library="SparkFun-PowerSymbols" library_urn="urn:adsk.eagle:library:530" deviceset="VCC" device=""/>
 <part name="J16" library="UltraLibrarianParts" deviceset="10103592-0001LF-EK" device=""/>
 <part name="J3" library="SparkFun-Connectors" library_urn="urn:adsk.eagle:library:513" deviceset="CONN_03" device="LONGPADS" package3d_urn="urn:adsk.eagle:package:38068/1"/>
@@
 <attribute name="NAME" x="177.8" y="79.248" size="1.778" layer="95" font="vector"/>
 </instance>
-<instance part="GND52" gate="1" x="208.28" y="53.34" smashed="yes">
-<attribute name="VALUE" x="208.28" y="53.086" size="1.778" layer="96" align="top-center"/>
-</instance>
-<instance part="SUPPLY20" gate="G$1" x="208.28" y="81.28" smashed="yes">
-<attribute name="VALUE" x="208.28" y="84.074" size="1.778" layer="96" align="bottom-center"/>
-</instance>
 </instances>
 <busses>
@@
 </segment>
 <segment>
-<pinref part="J15" gate="G$1" pin="6"/>
-<wire x1="187.96" y1="73.66" x2="208.28" y2="73.66" width="0.1524" layer="91"/>
-<wire x1="208.28" y1="73.66" x2="208.28" y2="55.88" width="0.1524" layer="91"/>
-<pinref part="GND52" gate="1" pin="GND"/>
+<pinref part="J15" gate="G$1" pin="5"/>
+<wire x1="187.96" y1="71.12" x2="190.5" y2="71.12" width="0.1524" layer="91"/>
+<label x="190.5" y="71.12" size="1.27" layer="95" xref="yes"/>
 </segment>
 </net>
@@
 </segment>
 <segment>
-<pinref part="J15" gate="G$1" pin="7"/>
-<wire x1="187.96" y1="76.2" x2="208.28" y2="76.2" width="0.1524" layer="91"/>
-<wire x1="208.28" y1="76.2" x2="208.28" y2="81.28" width="0.1524" layer="91"/>
-<pinref part="SUPPLY20" gate="G$1" pin="VCC"/>
+<pinref part="J15" gate="G$1" pin="3"/>
+<wire x1="187.96" y1="66.04" x2="190.5" y2="66.04" width="0.1524" layer="91"/>
+<label x="190.5" y="66.04" size="1.27" layer="95" xref="yes"/>
 </segment>
 </net>
@@
 </segment>
 <segment>
-<pinref part="J15" gate="G$1" pin="2"/>
-<wire x1="187.96" y1="63.5" x2="190.5" y2="63.5" width="0.1524" layer="91"/>
-<label x="190.5" y="63.5" size="1.27" layer="95" xref="yes"/>
+<pinref part="J15" gate="G$1" pin="6"/>
+<wire x1="187.96" y1="73.66" x2="190.5" y2="73.66" width="0.1524" layer="91"/>
+<label x="190.5" y="73.66" size="1.27" layer="95" xref="yes"/>
 </segment>
 </net>
@@
 </segment>
 <segment>
-<pinref part="J15" gate="G$1" pin="3"/>
-<wire x1="187.96" y1="66.04" x2="190.5" y2="66.04" width="0.1524" layer="91"/>
-<label x="190.5" y="66.04" size="1.27" layer="95" xref="yes"/>
+<pinref part="J15" gate="G$1" pin="2"/>
+<wire x1="187.96" y1="63.5" x2="190.5" y2="63.5" width="0.1524" layer="91"/>
+<label x="190.5" y="63.5" size="1.27" layer="95" xref="yes"/>
 </segment>
 </net>
@@
 </segment>
 <segment>
-<pinref part="J15" gate="G$1" pin="5"/>
-<wire x1="187.96" y1="71.12" x2="190.5" y2="71.12" width="0.1524" layer="91"/>
-<label x="190.5" y="71.12" size="1.27" layer="95" xref="yes"/>
+<pinref part="J15" gate="G$1" pin="1"/>
+<wire x1="187.96" y1="60.96" x2="190.5" y2="60.96" width="0.1524" layer="91"/>
+<label x="190.5" y="60.96" size="1.27" layer="95" xref="yes"/>
 </segment>
 </net>
@@
 </segment>
 </net>
-<net name="CD" class="0">
-<segment>
-<pinref part="J14" gate="A" pin="CD"/>
-<wire x1="205.74" y1="129.54" x2="215.9" y2="129.54" width="0.1524" layer="91"/>
-<label x="218.44" y="129.54" size="1.27" layer="95" xref="yes"/>
-<wire x1="215.9" y1="129.54" x2="218.44" y2="129.54" width="0.1524" layer="91"/>
-<wire x1="215.9" y1="129.54" x2="215.9" y2="132.08" width="0.1524" layer="91"/>
-<junction x="215.9" y="129.54"/>
-<wire x1="215.9" y1="132.08" x2="228.6" y2="132.08" width="0.1524" layer="91"/>
-<pinref part="R33" gate="G$1" pin="2"/>
-</segment>
-<segment>
-<pinref part="J15" gate="G$1" pin="1"/>
-<wire x1="187.96" y1="60.96" x2="190.5" y2="60.96" width="0.1524" layer="91"/>
-<label x="190.5" y="60.96" size="1.27" layer="95" xref="yes"/>
-</segment>
-</net>
 <net name="I2C_SCL" class="0">
 <segment>
@@
 </segment>
 </net>
+<net name="SPI_CD" class="0">
+<segment>
+<pinref part="J14" gate="A" pin="CD"/>
+<wire x1="205.74" y1="129.54" x2="215.9" y2="129.54" width="0.1524" layer="91"/>
+<label x="218.44" y="129.54" size="1.27" layer="95" xref="yes"/>
+<wire x1="215.9" y1="129.54" x2="218.44" y2="129.54" width="0.1524" layer="91"/>
+<wire x1="215.9" y1="129.54" x2="215.9" y2="132.08" width="0.1524" layer="91"/>
+<junction x="215.9" y="129.54"/>
+<wire x1="215.9" y1="132.08" x2="228.6" y2="132.08" width="0.1524" layer="91"/>
+<pinref part="R33" gate="G$1" pin="2"/>
+</segment>
+<segment>
+<pinref part="J15" gate="G$1" pin="7"/>
+<wire x1="187.96" y1="76.2" x2="190.5" y2="76.2" width="0.1524" layer="91"/>
+<label x="190.5" y="76.2" size="1.27" layer="95" xref="yes"/>
+</segment>
+</net>
