File: esp32/kitchensink_mini_esp32_v1.2.sch (EAGLE design)
At the start: 112 parts, among them J14 MEM2075-00-140-01-A, J16 10103592-0001LF-EK, J19 PJ-102AH, Q1 MMBT3904_R1, Q2 MMBT3904_R1, Q3 AO3401, Q4 PN2222A-SOT-23, U1 ESP32-WROOM-32D, U11 DS3231M+TRL21-0042B_16_MXM-M, U2 AP2111H-3.3TRG1SOT-223_DIO-M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

Commit message: Latest revision of kitchen sink mini v1.2
Connections:
- removed net N$32: C21.2, U9.IN
- removed net N$43: C21.1, D14.1
- new net N$14: C21.2, D14.1, U9.IN
- net GND: now also C21.1
Other:
- moved on the sheet: C21
Changed lines of the file:
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@@
 <part name="R12" library="standardparts" deviceset="RESISTOR" device=".1206" value="1K"/>
 <part name="GND17" library="SparkFun-PowerSymbols" library_urn="urn:adsk.eagle:library:530" deviceset="GND" device=""/>
+<part name="GND6" library="SparkFun-PowerSymbols" library_urn="urn:adsk.eagle:library:530" deviceset="GND" device=""/>
 </parts>
 <sheets>
@@
 <attribute name="VALUE" x="78.7386" y="50.7973" size="1.77848125" layer="96"/>
 </instance>
-<instance part="C21" gate="G$1" x="66.04" y="60.96" smashed="yes">
-<attribute name="NAME" x="64.77" y="62.865" size="1.016" layer="95" rot="MR90"/>
-<attribute name="VALUE" x="67.31" y="62.865" size="1.016" layer="96" rot="R90"/>
+<instance part="C21" gate="G$1" x="66.04" y="53.34" smashed="yes" rot="R90">
+<attribute name="NAME" x="64.135" y="52.07" size="1.016" layer="95" rot="MR0"/>
+<attribute name="VALUE" x="64.135" y="54.61" size="1.016" layer="96" rot="R180"/>
 </instance>
 <instance part="C22" gate="G$1" x="119.38" y="55.88" smashed="yes" rot="R90">
@@
 <instance part="TP67" gate="G$1" x="134.62" y="68.58" smashed="yes" rot="R90">
 <attribute name="NAME" x="137.16" y="66.04" size="1.778" layer="95" font="vector" rot="R90"/>
+</instance>
+<instance part="GND6" gate="1" x="66.04" y="40.64" smashed="yes">
+<attribute name="VALUE" x="66.04" y="40.386" size="1.778" layer="96" align="top-center"/>
 </instance>
 </instances>
@@
 <pinref part="GND62" gate="1" pin="GND"/>
 <wire x1="129.54" y1="48.26" x2="129.54" y2="43.18" width="0.1524" layer="91"/>
+</segment>
+<segment>
+<pinref part="C21" gate="G$1" pin="1"/>
+<pinref part="GND6" gate="1" pin="GND"/>
+<wire x1="66.04" y1="50.8" x2="66.04" y2="43.18" width="0.1524" layer="91"/>
 </segment>
 </net>
@@
 </segment>
 </net>
-<net name="N$32" class="0">
-<segment>
-<pinref part="U9" gate="G$1" pin="IN"/>
-<pinref part="C21" gate="G$1" pin="2"/>
-<wire x1="73.66" y1="60.96" x2="68.58" y2="60.96" width="0.1524" layer="91"/>
-</segment>
-</net>
 <net name="DC_JACK" class="1">
 <segment>
@@
 <wire x1="38.1" y1="68.58" x2="38.1" y2="60.96" width="0.1524" layer="91"/>
 <junction x="38.1" y="60.96"/>
-</segment>
-</net>
-<net name="N$43" class="0">
-<segment>
-<pinref part="C21" gate="G$1" pin="1"/>
-<pinref part="D14" gate="A" pin="1"/>
-<wire x1="55.88" y1="60.96" x2="63.5" y2="60.96" width="0.1524" layer="91"/>
 </segment>
 </net>
@@
 </segment>
 </net>
+<net name="N$14" class="0">
+<segment>
+<pinref part="D14" gate="A" pin="1"/>
+<pinref part="U9" gate="G$1" pin="IN"/>
+<wire x1="55.88" y1="60.96" x2="66.04" y2="60.96" width="0.1524" layer="91"/>
+<pinref part="C21" gate="G$1" pin="2"/>
+<wire x1="66.04" y1="60.96" x2="73.66" y2="60.96" width="0.1524" layer="91"/>
+<wire x1="66.04" y1="55.88" x2="66.04" y2="60.96" width="0.1524" layer="91"/>
+<junction x="66.04" y="60.96"/>
+</segment>
+</net>
